Commit message: ajout urdf

File: src/lerobot/configs/so100_minimal.urdf (robot description, URDF)
Before this commit: robot so100_arm, 7 links, 6 joints
Links:
- removed link base_link
- removed link elbow_link
- removed link gripper_frame_link
- removed link shoulder_lift_link
- removed link shoulder_pan_link
- removed link wrist_flex_link
- removed link wrist_roll_link
- added link base, mass 1.0; collision mesh filename=assets/Base.stl; visual mesh filename=assets/Base.stl
- added link gripper, mass 0.0929859; visual mesh filename=assets/Fixed_Jaw.stl; visual mesh filename=assets/Fixed_Jaw_Motor.stl
- added link jaw, mass 0.0202444; visual mesh filename=assets/Moving_Jaw.stl
- added link lower_arm, mass 0.147968; collision mesh filename=assets/Lower_Arm.stl; visual mesh filename=assets/Lower_Arm.stl
- added link shoulder, mass 0.119226; collision mesh filename=assets/Rotation_Pitch.stl; visual mesh filename=assets/Rotation_Pitch.stl
- added link upper_arm, mass 0.162409; collision mesh filename=assets/Upper_Arm.stl; visual mesh filename=assets/Upper_Arm.stl
- added link wrist, mass 0.0661321; collision mesh filename=assets/Wrist_Pitch_Roll.stl; visual mesh filename=assets/Wrist_Pitch_Roll.stl
Joints:
- removed joint elbow_flex_joint
- removed joint gripper_joint
- removed joint shoulder_lift_joint
- removed joint shoulder_pan_joint
- removed joint wrist_flex_joint
- removed joint wrist_roll_joint
- added joint elbow_flex: type revolute, parent upper_arm, child lower_arm, origin xyz=0 0.11257 0.028 rpy=1.57079 0 0, axis 1 0 0, limit lower=-3.14158 upper=0 effort=35 velocity=1
- added joint gripper: type revolute, parent gripper, child jaw, origin xyz=-0.0202 -0.0244 0 rpy=0 3.14158 0, axis 0 0 1, limit lower=-0.2 upper=2.0 effort=35 velocity=1
- added joint shoulder_lift: type revolute, parent shoulder, child upper_arm, origin xyz=0 0.1025 0.0306 rpy=-1.8 0 0, axis 1 0 0, limit lower=0 upper=3.5 effort=35 velocity=1
- added joint shoulder_pan: type revolute, parent base, child shoulder, origin xyz=0 -0.0452 0.0165 rpy=1.57079 0 0, axis 0 1 0, limit lower=-2 upper=2 effort=35 velocity=1
- added joint wrist_flex: type revolute, parent lower_arm, child wrist, origin xyz=0 0.0052 0.1349 rpy=-1 0 0, axis 1 0 0, limit lower=-2.5 upper=1.2 effort=35 velocity=1
- added joint wrist_roll: type revolute, parent wrist, child gripper, origin xyz=0 -0.0601 0 rpy=0 1.57079 0, axis 0 1 0, limit lower=-3.14158 upper=3.14158 effort=35 velocity=1
