Commit message: urdf

File: SO-ARM100/Simulation/SO100/so100.urdf (robot description, URDF)
Before this commit: robot so_arm100, 7 links, 6 joints
Links:
- added link gripper_frame_link
Joints:
- added joint gripper_to_frame: type fixed, parent jaw, child gripper_frame_link, origin xyz=0 0 0.05 rpy=0 0 0
